File: lib/Atmega328-GPIO.kicad_blocks/ARDU_RF_I2C.kicad_block/ARDU_RF_I2C.kicad_sch (KiCad schematic)
At the start: 5 parts, among them U1 NRF24L01_Breakout, U2 DHT11

Commit message: 5/21/25-1
Parts:
- added J12: Conn_01x04_Socket, Add_New:CONN_PPPC041LGBN-RC_SUL, symbol Connector:Conn_01x04_Socket
- added J4: Conn_01x04_Socket, Add_New:CONN_PPTC041LFBN-RC_SUL, symbol Connector:Conn_01x04_Socket
- added R13, R14: 10K, Resistor_THT:R_Axial_DIN0207_L6.3mm_D2.5mm_P10.16mm_Horizontal, symbol Device:R_US
- R15: footprint Resistor_THT:R_Axial_DIN0204_L3.6mm_D1.6mm_P5.08mm_Horizontal -> Resistor_THT:R_Axial_DIN0207_L6.3mm_D2.5mm_P10.16mm_Horizontal
Connections:
- net GND1: now also J12.4 (Pin_4), J4.3 (Pin_3), R13.2, R14.2
- net SCL1: now also J12.1 (Pin_1), J4.1 (Pin_1), R13.1
- net SDA1: now also J12.2 (Pin_2), J4.2 (Pin_2), R14.1
- net VCC1: now also J12.3 (Pin_3), J4.4 (Pin_4)
- net at A1.11 (D8): now also D8.2 (A)
- net at A1.5 (D2): no longer D8.2 (A)
- net 3V3 renamed 3V31
Other:
- note added: "I2C 16X2 LCD"
- note added: "I2C IO TEST"
- moved on the sheet: D8, R15
