File: lib/Atmega328-GPIO.kicad_blocks/I2C_LCD.kicad_block/I2C_LCD.kicad_sch (KiCad schematic)
At the start: 3 parts, among them J14 Conn_01x04_Socket

Commit message: 5/21/25-1
Parts:
- removed J14: Conn_01x04_Socket, Connector_Samtec_HPM_THT:Samtec_HPM-04-01-x-S_Straight_1x04_Pitch5.08mm, symbol Connector:Conn_01x04_Socket
- removed R49, R50: 10K, Resistor_THT:R_Axial_DIN0204_L3.6mm_D1.6mm_P5.08mm_Horizontal, symbol Device:R_US
- added J12: Conn_01x04_Socket, Add_New:CONN_PPPC041LGBN-RC_SUL, symbol Connector:Conn_01x04_Socket
Connections:
- new net GND1: J12.4 (Pin_4)
- new net SCL1: J12.1 (Pin_1)
- new net SDA1: J12.2 (Pin_2)
- new net VCC1: J12.3 (Pin_3)
Other:
- note added: "I2C 16X2 LCD"
- note removed: "I2C IO TEST"
